File: i2c-16c-demux.kicad_pcb (KiCad board)
At the start: 4 copper layers, 26 x 47 mm, 27 parts, among them J1 Conn_01x04, J2 Conn_01x04, J3 Conn_01x04, J4 Conn_01x04, J5 Conn_01x04, J6 Conn_01x02, Q1 CSD13380F3, Q10 CSD13380F3, Q11 CSD13380F3, Q12 CSD13380F3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

Commit message: PCB v1.2
Parts:
- JP_A0, JP_A1, JP_A2, U1: moved to B.Cu
- moved J2 102.8 mm to (120.7, 123.2), turned to 180 degrees
- moved Q1 93.9 mm to (126.9, 123.2), turned to 90 degrees
- moved J6 92.4 mm to (140.9, 124.5), turned to -90 degrees
- moved J3 91.6 mm to (120.7, 113.0), turned to 180 degrees
- moved Q2 90.3 mm to (130.8, 120.7), turned to 90 degrees
- moved Q3 87.4 mm to (126.9, 118.1), turned to 90 degrees
- moved Q4 84.1 mm to (130.8, 115.6), turned to 90 degrees
- moved Q5 81.6 mm to (126.9, 113.0), turned to 90 degrees
- moved Q6 78.6 mm to (130.8, 110.5), turned to 90 degrees
- moved JP_A2 78.5 mm to (132.7, 124.7), turned to 180 degrees
- moved Q7 76.5 mm to (126.9, 108.0), turned to 90 degrees
- moved JP_A0 75.4 mm to (146.7, 124.5), turned to 180 degrees
- moved JP_A1 74.0 mm to (139.7, 121.3), turned to 180 degrees
- moved Q8 73.9 mm to (130.8, 105.4), turned to 90 degrees
- moved U1 60.2 mm to (139.7, 114.3)
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Routing:
- net /OUT_1: track 46.5 -> 6.93 mm, vias 2 -> 0
- net /OUT_0: track 47.2 -> 9.65 mm, vias 3 -> 2
- net /OUT_3: track 38.5 -> 4.39 mm, vias 2 -> 0
- net /OUT_2: track 38.9 -> 8.60 mm
- net /OUT_5: track 32.8 -> 3.21 mm, vias 2 -> 0
- net /OUT_4: track 32.2 -> 7.55 mm
- net /OUT_7: track 27.7 -> 4.00 mm, vias 2 -> 0
- net /OUT_6: track 27.4 -> 7.29 mm
- net Net-(U1-P1): track 24.4 -> 8.47 mm, vias 2 -> 1
- net Net-(U1-P0): track 21.7 -> 6.88 mm, vias 2 -> 1
- net Net-(U1-P5): track 25.1 -> 10.9 mm, vias 2 -> 1
- net Net-(U1-P2): track 22.7 -> 9.84 mm, vias 2 -> 1
- net /A1: track 17.2 -> 4.74 mm, vias 2 -> 0
- net /A0: track 21.7 -> 9.36 mm, vias 2 -> 0
- net Net-(U1-P4): track 16.5 -> 5.04 mm, vias 2 -> 1
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Other:
- board size 26 x 47 mm -> 41.9 x 25.4 mm
- board text added: "G0"
- board text added: "G1"
- board text added: "G2"
- board text added: "G3"
- board text added: "G4"
- board text added: "G5"
- board text added: "G6"
- board text added: "G7"
- board text added: "G8"
- board text added: "G9"
- board text added: "Ga"
- board text added: "Gb"
- board text added: "Gc"
- board text added: "Gd"
- board text added: "Ge"
- board text added: "Gf"
